Commit message: Add files via upload

File: src/my_robot_description/urdf/common_properties.xacro (robot description, xacro)
@@ -3,4 +3,10 @@
     <material name = "green">
         <color rgba = "0 0.5 0 1" />
+    </material>
+    <material name = "orange">
+        <color rgba = "1 0.5 0 1" />
+    </material>
+    <material name = "yellow">
+        <color rgba = "1 1 0 1" />
     </material>
     <material name = "blue">
