Commit message: Add files via upload

File: src/my_robot_description/urdf/arm.xacro (robot description, xacro)
@@ -22,5 +22,5 @@
             <origin xyz = "0 0 ${arm_base_height / 2.0}" rpy = "0 0 0" />
         </collision>
-        <xacro:box_inertia m = "0.5" l = "${3*arm_base_length}" w = "${3*arm_base_width}" h = "${3*arm_base_height}"
+        <xacro:box_inertia m = "0.5" l = "${4*arm_base_length}" w = "${4*arm_base_width}" h = "${4*arm_base_height}"
                            xyz = "0 0 ${arm_base_height / 2.0}" rpy = "0 0 0" />
     </link>
@@ -39,5 +39,5 @@
             <origin xyz = "0 0 ${forearm_length / 2.0}" rpy = "0 0 0" />
         </collision>
-        <xacro:wheel_inertia m = "0.3" r = "${3*forearm_radius}" l = "${3*forearm_length}"
+        <xacro:wheel_inertia m = "0.3" r = "${4*forearm_radius}" l = "${4*forearm_length}"
                              xyz = "0 0 ${forearm_length / 2.0}" rpy = "0 0 0" />
     </link>
@@ -56,5 +56,5 @@
             <origin xyz = "0 0 ${hand_length / 2.0}" rpy = "0 0 0" />
         </collision>
-        <xacro:wheel_inertia m = "0.3" r = "${3*hand_radius}" l = "${3*hand_length}"
+        <xacro:wheel_inertia m = "0.3" r = "${4*hand_radius}" l = "${4*hand_length}"
                              xyz = "0 0 ${hand_length / 2.0}" rpy = "0 0 0" />
     </link>

File: src/my_robot_description/urdf/arm_gazebo.xacro (robot description, xacro)
@@ -1,12 +1,29 @@
 <?xml version = "1.0"?>
 <robot xmlns:xacro = "http://www.ros.org/wiki/xacro">
-<gazebo reference = "arm_base_link">
-    <material>Gazebo/Orange</material>
-</gazebo>
-<gazebo reference = "forearm_link">
-    <material>Gazebo/Yellow</material>
-</gazebo>
-<gazebo reference = "hand_link">
-    <material>Gazebo/Orange</material>
-</gazebo>
+    <gazebo reference = "arm_base_link">
+        <material>Gazebo/Orange</material>
+    </gazebo>
+    <gazebo reference = "forearm_link">
+        <material>Gazebo/Yellow</material>
+    </gazebo>
+    <gazebo reference = "hand_link">
+        <material>Gazebo/Orange</material>
+    </gazebo>
+    <gazebo>
+        <plugin name = "joint_state_publisher_controller"
+                filename = "libgazebo_ros_joint_state_publisher.so">
+            <!-- <update rate in hertz> -->
+            <update_rate>10</update_rate>
+            <!-- <Name of the joint in the model whose state will be published> -->
+            <joint_name>arm_base_forearm_joint</joint_name>
+            <joint_name>forearm_hand_joint</joint_name>
+        </plugin>
+    </gazebo>
+    <gazebo>
+        <plugin name = "joint_pose_trajectory_controller"
+                filename = "libgazebo_ros_joint_pose_trajectory.so">
+            <!-- <update rate in hertz> -->
+            <update_rate>2</update_rate>
+        </plugin>
+    </gazebo>
 </robot>

File: src/my_robot_description/urdf/my_robot.urdf.xacro (robot description, xacro)
@@ -4,4 +4,11 @@
     <xacro:include filename = "mobile_base.xacro" />
     <xacro:include filename = "mobile_base_gazebo.xacro" />
-    <xacro:include filename = "camera.xacro" />
+    <xacro:include filename = "arm.xacro" />
+    <xacro:include filename = "arm_gazebo.xacro" />
+    <!-- <xacro:include filename = "camera.xacro" /> -->
+    <joint name = "mobile_base_arm_joint" type = "fixed">
+        <parent link = "base_link" />
+        <child link = "arm_base_link" />
+        <origin xyz = "${base_length / 4.0} 0 ${base_height}" rpy = "0 0 0" />
+    </joint>
 </robot>
