Commit message: Add files via upload

File: src/my_robot_description/urdf/my_robot.urdf.xacro (robot description, xacro)
@@ -4,11 +4,12 @@
     <xacro:include filename = "mobile_base.xacro" />
     <xacro:include filename = "mobile_base_gazebo.xacro" />
-    <xacro:include filename = "arm.xacro" />
-    <xacro:include filename = "arm_gazebo.xacro" />
+    <!-- <xacro:include filename = "arm.xacro" />
+    <xacro:include filename = "arm_gazebo.xacro" /> -->
     <!-- <xacro:include filename = "camera.xacro" /> -->
-    <joint name = "mobile_base_arm_joint" type = "fixed">
+    <xacro:include filename = "lidar.xacro" />
+    <!-- <joint name = "mobile_base_arm_joint" type = "fixed">
         <parent link = "base_link" />
         <child link = "arm_base_link" />
         <origin xyz = "${base_length / 4.0} 0 ${base_height}" rpy = "0 0 0" />
-    </joint>
+    </joint> -->
 </robot>
